Commit message: Add green back plate
This update to "hexagons1.urdf.xacro" adds a link modeling a plate which is configured to be green and attached to the top plate of the Turtlebot. It allows performing a simple thresholding-based following behavior.

File: turtlebot/turtlebot_description/urdf/stacks/hexagons1.urdf.xacro (robot description, xacro)
@@ -223,4 +223,36 @@
       </inertial>
     </link>
+    <!-- Green plate that will be attached at the back of the Turtlebot -->
+    <link name="back_green_plate">
+      <visual>
+        <origin xyz="0 0 0" rpy="0 0 0"/>
+        <geometry>
+	  <box size="0.01 0.21 0.30"/>
+        </geometry>
+      </visual>
+      <collision>
+        <origin xyz="0 0 0" rpy="0 0 0"/>
+        <geometry>
+	  <box size="0.01 0.21 0.30"/>
+        </geometry>
+      </collision>
+      <inertial>
+        <mass value="0.005"/>
+        <origin xyz="0 0 0"/>
+        <inertia ixx="0.003328" ixy="0.0" ixz="0.0"
+                 iyy="0.003328" iyz="0.0"
+                 izz="0.006656" />
+      </inertial>
+    </link>
+    <!-- Set green color for the back plate -->
+    <gazebo reference="back_green_plate">
+      <material>Gazebo/Green</material>
+    </gazebo>
+    <!-- Add the back plate to the model (w a fixed joint) -->
+    <joint name="back_plate_joint" type="fixed">
+      <parent link="plate_top_link"/>
+      <child link="back_green_plate"/>
+      <origin xyz="-0.15 0 -0.15" rpy="0 0 0"/>
+    </joint>
   </xacro:macro>
 </robot>
